Commit message: multirobot_add

File: husky_description/urdf/decorations.urdf.xacro (robot description, xacro)
@@ -8,9 +8,9 @@
   <material name="white"><color rgba="1.0 1.0 1.0 1.0" /></material>
   <material name="red"><color rgba="1.0 0.0 0.0 1.0" /></material>
-  <xacro:macro name="husky_decorate">
+  <xacro:macro name="husky_decorate" params="prefix">
     <xacro:property name="husky_front_bumper_extend" value="$(optenv HUSKY_FRONT_BUMPER_EXTEND 0)" />
     <xacro:property name="husky_rear_bumper_extend" value="$(optenv HUSKY_REAR_BUMPER_EXTEND 0)" />
     <!-- Spawn Husky chassis -->
-    <link name="top_chassis_link">
+    <link name="${prefix}top_chassis_link">
       <visual>
         <origin xyz="0 0 0" rpy="0 0 0" />
@@ -21,11 +21,11 @@
     </link>
     <!-- Attach chassis to the robot -->
-    <joint name="top_chassis_joint" type="fixed">
-      <parent link="base_link" />
-      <child link="top_chassis_link" />
+    <joint name="${prefix}top_chassis_joint" type="fixed">
+      <parent link="${prefix}base_link" />
+      <child link="${prefix}top_chassis_link" />
     </joint>
     <xacro:if value="$(optenv HUSKY_USER_RAIL_ENABLED true)">
       <!-- Spawn user rails -->
-      <link name="user_rail_link">
+      <link name="${prefix}user_rail_link">
         <visual>
           <geometry>
@@ -35,12 +35,12 @@
       </link>
       <!-- Attach user rails to base link -->
-      <joint name="user_rail" type="fixed">
+      <joint name="${prefix}user_rail" type="fixed">
         <origin xyz="0.272 0 0.245" rpy="0 0 0" />
-        <parent link="base_link" />
-        <child link="user_rail_link" />
+        <parent link="${prefix}base_link" />
+        <child link="${prefix}user_rail_link" />
       </joint>
     </xacro:if>
     <!-- Spawn front bumper link -->
-    <link name="front_bumper_link">
+    <link name="${prefix}front_bumper_link">
       <visual>
         <geometry>
@@ -50,11 +50,11 @@
     </link>
     <!-- Attach front bumper -->
-    <joint name="front_bumper" type="fixed">
+    <joint name="${prefix}front_bumper" type="fixed">
       <origin xyz="${0.48 + husky_front_bumper_extend} 0 0.091" rpy="0 0 0" />
-      <parent link="base_link" />
-      <child link="front_bumper_link" />
+      <parent link="${prefix}base_link" />
+      <child link="${prefix}front_bumper_link" />
     </joint>
     <xacro:if value="${husky_front_bumper_extend}">
-      <link name="front_bumper_extension_link">
+      <link name="${prefix}front_bumper_extension_link">
           <visual>
               <geometry>
@@ -63,12 +63,12 @@
           </visual>
       </link>
-      <joint name="front_bumper_extension" type="fixed">
+      <joint name="${prefix}front_bumper_extension" type="fixed">
         <origin xyz="${0.48 + husky_front_bumper_extend} 0 0.091" rpy="0 0 0" />
-        <parent link="base_link" />
-        <child link="front_bumper_extension_link" />
+        <parent link="${prefix}base_link" />
+        <child link="${prefix}front_bumper_extension_link" />
       </joint>
     </xacro:if>
     <!-- Spawn rear bumper link -->
-    <link name="rear_bumper_link">
+    <link name="${prefix}rear_bumper_link">
       <visual>
         <geometry>
@@ -78,11 +78,11 @@
     </link>
     <!-- Attach rear bumper -->
-    <joint name="rear_bumper" type="fixed">
+    <joint name="${prefix}rear_bumper" type="fixed">
       <origin xyz="${-0.48 - husky_rear_bumper_extend} 0 0.091" rpy="0 0 ${M_PI}" />
-      <parent link="base_link" />
-      <child link="rear_bumper_link" />
+      <parent link="${prefix}base_link" />
+      <child link="${prefix}rear_bumper_link" />
     </joint>
     <xacro:if value="${husky_rear_bumper_extend}">
-      <link name="rear_bumper_extension_link">
+      <link name="${prefix}rear_bumper_extension_link">
           <visual>
               <geometry>
@@ -91,8 +91,8 @@
           </visual>
       </link>
-      <joint name="rear_bumper_extension" type="fixed">
+      <joint name="${prefix}rear_bumper_extension" type="fixed">
         <origin xyz="${-0.48 - husky_rear_bumper_extend} 0 0.091" rpy="0 0 ${M_PI}" />
-        <parent link="base_link" />
-        <child link="rear_bumper_extension_link" />
+        <parent link="${prefix}base_link" />
+        <child link="${prefix}rear_bumper_extension_link" />
       </joint>
     </xacro:if>
@@ -100,5 +100,5 @@
       <!-- Spawn the top plate -->
       <xacro:if value="$(optenv HUSKY_LARGE_TOP_PLATE false)">
-        <link name="top_plate_link">
+        <link name="${prefix}top_plate_link">
           <visual>
             <origin xyz="0 0 0" rpy="0 0 0" />
@@ -115,24 +115,24 @@
         </link>
         <!-- Attach top plate -->
-        <joint name="top_plate_joint" type="fixed">
-          <parent link="base_link" />
-          <child link="top_plate_link"/>
+        <joint name="${prefix}top_plate_joint" type="fixed">
+          <parent link="${prefix}base_link" />
+          <child link="${prefix}top_plate_link"/>
           <origin xyz="0.0812 0 0.225" rpy="0 0 0"/>
         </joint>
         <!-- Top plate front link -->
-        <joint name="top_plate_front_joint" type="fixed">
-          <parent link="top_plate_link" />
-          <child link="top_plate_front_link"/>
+        <joint name="${prefix}top_plate_front_joint" type="fixed">
+          <parent link="${prefix}top_plate_link" />
+          <child link="${prefix}top_plate_front_link"/>
           <origin xyz="0.4125 0 0.00672" rpy="0 0 0"/>
         </joint>
         <!-- Top plate rear link-->
-        <joint name="top_plate_rear_joint" type="fixed">
-          <parent link="top_plate_link" />
-          <child link="top_plate_rear_link"/>
+        <joint name="${prefix}top_plate_rear_joint" type="fixed">
+          <parent link="${prefix}top_plate_link" />
+          <child link="${prefix}top_plate_rear_link"/>
           <origin xyz="-0.4125 0 0.00672" rpy="0 0 0"/>
         </joint>
       </xacro:if>
       <xacro:unless value="$(optenv HUSKY_LARGE_TOP_PLATE false)">
-        <link name="top_plate_link">
+        <link name="${prefix}top_plate_link">
           <visual>
             <origin xyz="0 0 0" rpy="0 0 0" />
@@ -149,24 +149,24 @@
         </link>
         <!-- Attach top plate -->
-        <joint name="top_plate_joint" type="fixed">
-          <parent link="base_link" />
-          <child link="top_plate_link"/>
+        <joint name="${prefix}top_plate_joint" type="fixed">
+          <parent link="${prefix}base_link" />
+          <child link="${prefix}top_plate_link"/>
           <origin xyz="0.0812 0 0.245" rpy="0 0 0"/>
         </joint>
         <!-- Top plate front link -->
-        <joint name="top_plate_front_joint" type="fixed">
-          <parent link="top_plate_link" />
-          <child link="top_plate_front_link"/>
+        <joint name="${prefix}top_plate_front_joint" type="fixed">
+          <parent link="${prefix}top_plate_link" />
+          <child link="${prefix}top_plate_front_link"/>
           <origin xyz="0.36367 0 0.00639" rpy="0 0 0"/>
         </joint>
         <!-- Top plate rear link-->
-        <joint name="top_plate_rear_joint" type="fixed">
-          <parent link="top_plate_link" />
-          <child link="top_plate_rear_link"/>
+        <joint name="${prefix}top_plate_rear_joint" type="fixed">
+          <parent link="${prefix}top_plate_link" />
+          <child link="${prefix}top_plate_rear_link"/>
           <origin xyz="-0.36633 0 0.00639" rpy="0 0 0"/>
         </joint>
       </xacro:unless>
-      <link name="top_plate_front_link"/>
-      <link name="top_plate_rear_link"/>
+      <link name="${prefix}top_plate_front_link"/>
+      <link name="${prefix}top_plate_rear_link"/>
     </xacro:if>
   </xacro:macro>

File: husky_description/urdf/husky.urdf (no_ros2_control).xacro (robot description, xacro)
@@ -4,11 +4,14 @@
   <!-- <xacro:arg name="name" default="" /> -->
   <xacro:arg name="prefix" default="" />
-  <xacro:arg name="namespace" default="" />
   <xacro:arg name="gazebo_controllers" default="$(find husky_control)/config/control.yaml" />
   <xacro:include filename="$(find husky_description)/urdf/husky_macro.urdf.xacro" />
-  <xacro:include filename="$(find husky_description)/urdf/gazebo_control.xacro" />
   <!-- Load husky description -->
   <xacro:husky prefix="$(arg prefix)" />
   <xacro:if value="$(arg is_sim)">
+    <gazebo>
+      <plugin name="gazebo_ros2_control" filename="libgazebo_ros2_control.so">
+        <parameters>$(arg gazebo_controllers)</parameters>
+      </plugin>
+    </gazebo>
     <gazebo reference="imu_link">
       <sensor name="$(arg prefix)imu_sensor" type="imu">

File: husky_description/urdf/husky.urdf(save).xacro (robot description, xacro)
@@ -4,12 +4,15 @@
   <!-- <xacro:arg name="name" default="" /> -->
   <xacro:arg name="prefix" default="" />
-  <xacro:arg name="namespace" default="" />
   <xacro:arg name="gazebo_controllers" default="$(find husky_control)/config/control.yaml" />
   <xacro:include filename="$(find husky_description)/urdf/husky_macro.urdf.xacro" />
-  <xacro:include filename="$(find husky_description)/urdf/gazebo_control.xacro" />
   <!-- Load husky description -->
   <xacro:husky prefix="$(arg prefix)" />
   <xacro:if value="$(arg is_sim)">
-    <gazebo reference="imu_link">
+    <gazebo>
+      <plugin name="$(arg prefix)gazebo_ros2_control" filename="libgazebo_ros2_control.so">
+        <parameters>$(arg gazebo_controllers)</parameters>
+      </plugin>
+    </gazebo>
+    <gazebo reference="$(arg prefix)imu_link">
       <sensor name="$(arg prefix)imu_sensor" type="imu">
       <plugin filename="libgazebo_ros_imu_sensor.so" name="$(arg prefix)imu_plugin">
@@ -25,7 +28,7 @@
       </sensor>
     </gazebo>
-    <gazebo reference="$gps_link">
+    <gazebo reference="$(arg prefix)gps_link">
       <sensor name="$(arg prefix)gps_sensor" type="gps">
-      <plugin filename="libgazebo_ros_gps_sensor.so" name="gps_plugin">
+      <plugin filename="libgazebo_ros_gps_sensor.so" name="$(arg prefix)gps_plugin">
           <ros>
             <namespace>$(arg prefix)</namespace>

File: husky_description/urdf/husky_macro.urdf (save).xacro (robot description, xacro)
@@ -13,6 +13,7 @@
   <xacro:arg name="is_sim" default="false" />
   <xacro:arg name="urdf_extras" default="$(optenv CPR_URDF_EXTRAS empty.urdf)" />
+  <xacro:arg name="serial_port" default="$(optenv HUSKY_SERIAL_PORT /dev/prolific)" />
   <!-- Included URDF/XACRO Files -->
-  <xacro:include filename="$(find husky_description)/urdf/decorations.urdf.xacro" />
+  <!--xacro:include filename="$(find husky_description)/urdf/decorations.urdf.xacro" /-->
   <xacro:include filename="$(find husky_description)/urdf/wheel.urdf.xacro" />
   <xacro:include filename="$(find husky_description)/urdf/accessories/intel_realsense.urdf.xacro"/>
@@ -102,5 +103,5 @@
       <origin xyz="${-wheelbase/2} ${-track/2} ${wheel_vertical_offset}" rpy="0 0 0" />
     </xacro:husky_wheel>
-    <xacro:husky_decorate prefix="$(arg prefix)"/>
+    <!--xacro:husky_decorate /-->
     <!-- <xacro:if value="$(arg laser_enabled)">
       <xacro:sick_lms1xx_mount prefix="base"/>
@@ -146,6 +147,6 @@
           <param name="max_accel">5.0</param>
           <param name="max_speed">1.0</param>
-          <param name="polling_timeout">10.0</param>
-          <param name="serial_port">/dev/prolific</param>
+          <param name="polling_timeout">0.1</param>
+          <param name="serial_port">$(arg serial_port)</param>
         </xacro:unless>
       </hardware>

File: husky_description/urdf/wheel.urdf.xacro (robot description, xacro)
@@ -29,5 +29,5 @@
     </gazebo>
     <joint name="${wheel_prefix}_wheel_joint" type="continuous">
-      <parent link="base_link"/>
+      <parent link="${prefix}base_link"/>
       <child link="${wheel_prefix}_wheel"/>
       <xacro:insert_block name="joint_pose"/>
