Commit message: updates

File: husky_description/urdf/wheel.urdf.xacro (robot description, xacro)
@@ -17,5 +17,5 @@
         <origin xyz="0 0 0" rpy="${M_PI/2} 0 0" />
         <geometry>
-          <cylinder length="${wheel_length}" radius="${wheel_radius}" />
+          <cylinder length="${wheel_length+0.01}" radius="${wheel_radius+0.03}" />
         </geometry>
       </collision>
