Commit message: added laser_scan topics

File: husky_description/urdf/accessories/sick_lms1xx_mount.urdf.xacro (robot description, xacro)
@@ -26,5 +26,5 @@
 -->
 <robot xmlns:xacro="http://ros.org/wiki/xacro">
-  <xacro:include filename="$(find lms1xx)/urdf/sick_lms1xx.urdf.xacro" />
+  <xacro:include filename="$(find husky_description)/urdf/accessories/sick_lms1xx.urdf.xacro" />
   <xacro:macro name="sick_lms1xx_mount" params="prefix">
     <link name="${prefix}_laser_mount">

File: husky_description/urdf/husky.urdf.xacro (robot description, xacro)
@@ -10,4 +10,5 @@
   <!-- Load husky description -->
   <xacro:husky prefix="$(arg prefix)" />
+  <xacro:lidar prefix="$(arg prefix)" />
   <xacro:if value="$(arg is_sim)">
     <gazebo reference="$(arg prefix)imu_link">
@@ -37,4 +38,33 @@
       </sensor>
     </gazebo>
+    <gazebo reference="$(arg prefix)base_lidar">
+      <sensor name="$(arg prefix)lidar" type="ray">
+        <visualize>false</visualize>
+        <update_rate>10</update_rate>
+        <ray>
+          <scan>
+            <horizontal>
+              <samples>720</samples>
+              <resolution>1</resolution>
+              <min_angle>-1.8</min_angle>
+              <max_angle>1.8</max_angle>
+            </horizontal>
+          </scan>
+          <range>
+            <min>0.3</min>
+            <max>30.0</max>
+            <resolution>0.01</resolution>
+          </range>
+        </ray>
+        <plugin name="$(arg prefix)lidar" filename="libgazebo_ros_ray_sensor.so">
+          <output_type>sensor_msgs/LaserScan</output_type>
+          <ros>
+            <namespace>$(arg prefix)</namespace>
+            <remapping>~/out:=scan</remapping>
+          </ros>
+          <frame_name>$(arg prefix)base_lidar</frame_name>
+        </plugin>
+      </sensor>
+    </gazebo>
   </xacro:if>
   <!-- Optional custom includes. -->

File: husky_description/urdf/husky_macro.urdf (save).xacro (robot description, xacro)
@@ -20,13 +20,4 @@
   <xacro:include filename="$(find husky_description)/urdf/accessories/sensor_arch.urdf.xacro"/>
   <xacro:property name="M_PI" value="3.14159"/>
-  <!-- Husky Macro for lidar-->
-  <xacro:macro name="lidar" params="prefix">
-    <link name="${prefix}base_lidar"/>
-    <joint name="${prefix}base_lidar_joint" type="fixed">
-      <origin xyz="0.55 0 0.13" rpy="0 0 0" />
-      <parent link="${prefix}base_link" />
-      <child link="${prefix}base_lidar" />
-    </joint>
-  </xacro:macro>
   <xacro:macro name="husky" params="prefix">
     <!-- Base Size -->
